File: pcb/Hackpad_PCB_Gwendal_revB.kicad_pcb (KiCad board)
At the start: 2 copper layers, 100 x 100 mm, 50 parts, among them SW1 SW_Push, SW10 SW_Push, SW11 SW_Push, SW12 SW_Push, SW13 SW_Push, SW14 SW_Push, SW15 SW_Push, SW16 SW_Push, SW17 RotaryEncoder_Switch, SW18 RotaryEncoder_Switch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

Commit message: Edited Oled pullups to be 3.3v reference instead of 5v, I won't edit all of the pictures for such a small change.
Parts:
- SW1, SW10, SW11, SW12, SW13, SW14, SW15, SW16, SW2, SW3, SW4, SW5, SW6, SW7, SW8, SW9: footprint Alps_Solderable:SW_Cherry_MX_1.00u_PCB -> Button_Switch_Keyboard:SW_Cherry_MX_1.00u_PCB
Connections:
- R7 pad 1: VCC -> +3.3V
- R8 pad 1: VCC -> +3.3V
Routing:
- net +3.3V: track 105.5 -> 139.7 mm, vias 0 -> 1
- net VCC: track 42.6 -> 35.0 mm

Commit message: Added a copper fill zone to the front and back of the PCB.
Routing:
- added copper zone on B.Cu, net (none)
- added copper zone on F.Cu, net (none)
Changed lines of the file:
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@@
 		(net 41)
+	)
+	(zone
+		(net 0)
+		(net_name "")
+		(layers "F.Cu" "B.Cu")
+		(hatch edge 0.5)
+		(connect_pads
+			(clearance 0.5)
+		)
+		(min_thickness 0.25)
+		(filled_areas_thickness no)
+		(fill yes
+			(thermal_gap 0.5)
+			(thermal_bridge_width 0.5)
+			(island_removal_mode 1)
+			(island_area_min 10)
+		)
+		(polygon
+			(pts
+				(xy 82 33.5) (xy 81.5 137) (xy 186 136) (xy 185.5 32.5)
+			)
+		)
 	)
 	(group ""

Commit message: Updated "MADE IN RENNES" to "DESIGNED IN RENNES" on the pcb graphics, as JLCPCB failed the first audit because of it.
Routing:
- removed copper zone on B.Cu, net (none)
- removed copper zone on F.Cu, net (none)
